File: pcbs/reflow-controller-v1/display_lcd.kicad_sch (KiCad schematic)
At the start: 5 parts, among them J701 PinHeader 1x14 P2.54mm

Commit message: added temp sensor
Parts:
- renumbered H801 to H701, H801 to H702, H801 to H703, H801 to H704
Changed lines of the file:
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@@
   (symbol (lib_id "Mechanical:MountingHole_Pad") (at 215.9 81.28 0) (unit 1)
     (in_bom yes) (on_board yes) (dnp no) (fields_autoplaced)
-    (property "Reference" "H801" (at 218.44 78.74 0)
+    (property "Reference" "H702" (at 218.44 78.74 0)
       (effects (font (size 1.27 1.27)) (justify left))
     )
@@
     (instances
       (project "reflow-controller-v1"
-        (path "/843848ae-bf49-42cb-8f8b-76790d2e568d/41c2d982-496b-4922-a077-a2a7f833416c"
-          (reference "H801") (unit 1)
-        )
-        (path "/843848ae-bf49-42cb-8f8b-76790d2e568d/28d32604-417d-4cd4-a8ef-2fae619450e6"
-          (reference "H901") (unit 1)
-        )
         (path "/843848ae-bf49-42cb-8f8b-76790d2e568d/f628d05d-4e2a-4195-9ee3-f88b775e9255"
           (reference "H702") (unit 1)
@@
   (symbol (lib_id "Mechanical:MountingHole_Pad") (at 215.9 72.39 0) (unit 1)
     (in_bom yes) (on_board yes) (dnp no) (fields_autoplaced)
-    (property "Reference" "H801" (at 218.44 69.85 0)
+    (property "Reference" "H701" (at 218.44 69.85 0)
       (effects (font (size 1.27 1.27)) (justify left))
     )
@@
     (instances
       (project "reflow-controller-v1"
-        (path "/843848ae-bf49-42cb-8f8b-76790d2e568d/41c2d982-496b-4922-a077-a2a7f833416c"
-          (reference "H801") (unit 1)
-        )
-        (path "/843848ae-bf49-42cb-8f8b-76790d2e568d/28d32604-417d-4cd4-a8ef-2fae619450e6"
-          (reference "H901") (unit 1)
-        )
         (path "/843848ae-bf49-42cb-8f8b-76790d2e568d/f628d05d-4e2a-4195-9ee3-f88b775e9255"
           (reference "H701") (unit 1)
@@
   (symbol (lib_id "Mechanical:MountingHole_Pad") (at 215.9 90.17 0) (unit 1)
     (in_bom yes) (on_board yes) (dnp no) (fields_autoplaced)
-    (property "Reference" "H801" (at 218.44 87.63 0)
+    (property "Reference" "H703" (at 218.44 87.63 0)
       (effects (font (size 1.27 1.27)) (justify left))
     )
@@
     (instances
       (project "reflow-controller-v1"
-        (path "/843848ae-bf49-42cb-8f8b-76790d2e568d/41c2d982-496b-4922-a077-a2a7f833416c"
-          (reference "H801") (unit 1)
-        )
-        (path "/843848ae-bf49-42cb-8f8b-76790d2e568d/28d32604-417d-4cd4-a8ef-2fae619450e6"
-          (reference "H901") (unit 1)
-        )
         (path "/843848ae-bf49-42cb-8f8b-76790d2e568d/f628d05d-4e2a-4195-9ee3-f88b775e9255"
           (reference "H703") (unit 1)
@@
   (symbol (lib_id "Mechanical:MountingHole_Pad") (at 215.9 99.06 0) (unit 1)
     (in_bom yes) (on_board yes) (dnp no) (fields_autoplaced)
-    (property "Reference" "H801" (at 218.44 96.52 0)
+    (property "Reference" "H704" (at 218.44 96.52 0)
       (effects (font (size 1.27 1.27)) (justify left))
     )
@@
     (instances
       (project "reflow-controller-v1"
-        (path "/843848ae-bf49-42cb-8f8b-76790d2e568d/41c2d982-496b-4922-a077-a2a7f833416c"
-          (reference "H801") (unit 1)
-        )
-        (path "/843848ae-bf49-42cb-8f8b-76790d2e568d/28d32604-417d-4cd4-a8ef-2fae619450e6"
-          (reference "H901") (unit 1)
-        )
         (path "/843848ae-bf49-42cb-8f8b-76790d2e568d/f628d05d-4e2a-4195-9ee3-f88b775e9255"
           (reference "H704") (unit 1)

Commit message: footprint assignement fixed; buzzer added
Parts:
- H701, H702, H703, H704: value SMTSO2540CTJ -> SMTSO2040CTJ; footprint WA-SMSI_M2.5:Mounting_Wuerth_WA-SMSI-M2.5_H4mm_9774040151 -> Mounting_Wuerth:Mounting_Wuerth_WA-SMSI-M2_H4mm_9774040243
Changed lines of the file:
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@@
 		(fields_autoplaced yes)
 		(property "Reference" "H702"
-			(at 218.44 78.74 0)
-			(effects
-				(font
-					(size 1.27 1.27)
-				)
-				(justify left)
-			)
-		)
-		(property "Value" "SMTSO2540CTJ"
-			(at 218.44 81.28 0)
-			(effects
-				(font
-					(size 1.27 1.27)
-				)
-				(justify left)
-			)
-		)
-		(property "Footprint" "WA-SMSI_M2.5:Mounting_Wuerth_WA-SMSI-M2.5_H4mm_9774040151"
+			(at 218.44 78.7399 0)
+			(effects
+				(font
+					(size 1.27 1.27)
+				)
+				(justify left)
+			)
+		)
+		(property "Value" "SMTSO2040CTJ"
+			(at 218.44 81.2799 0)
+			(effects
+				(font
+					(size 1.27 1.27)
+				)
+				(justify left)
+			)
+		)
+		(property "Footprint" "Mounting_Wuerth:Mounting_Wuerth_WA-SMSI-M2_H4mm_9774040243"
 			(at 215.9 81.28 0)
 			(effects
@@
 			)
 		)
-		(property "Value" "SMTSO2540CTJ"
+		(property "Value" "SMTSO2040CTJ"
 			(at 218.44 72.39 0)
 			(effects
@@
 			)
 		)
-		(property "Footprint" "WA-SMSI_M2.5:Mounting_Wuerth_WA-SMSI-M2.5_H4mm_9774040151"
+		(property "Footprint" "Mounting_Wuerth:Mounting_Wuerth_WA-SMSI-M2_H4mm_9774040243"
 			(at 215.9 72.39 0)
 			(effects
@@
 		(fields_autoplaced yes)
 		(property "Reference" "H703"
-			(at 218.44 87.63 0)
-			(effects
-				(font
-					(size 1.27 1.27)
-				)
-				(justify left)
-			)
-		)
-		(property "Value" "SMTSO2540CTJ"
-			(at 218.44 90.17 0)
-			(effects
-				(font
-					(size 1.27 1.27)
-				)
-				(justify left)
-			)
-		)
-		(property "Footprint" "WA-SMSI_M2.5:Mounting_Wuerth_WA-SMSI-M2.5_H4mm_9774040151"
+			(at 218.44 87.6299 0)
+			(effects
+				(font
+					(size 1.27 1.27)
+				)
+				(justify left)
+			)
+		)
+		(property "Value" "SMTSO2040CTJ"
+			(at 218.44 90.1699 0)
+			(effects
+				(font
+					(size 1.27 1.27)
+				)
+				(justify left)
+			)
+		)
+		(property "Footprint" "Mounting_Wuerth:Mounting_Wuerth_WA-SMSI-M2_H4mm_9774040243"
 			(at 215.9 90.17 0)
 			(effects
@@
 		(fields_autoplaced yes)
 		(property "Reference" "H704"
-			(at 218.44 96.52 0)
-			(effects
-				(font
-					(size 1.27 1.27)
-				)
-				(justify left)
-			)
-		)
-		(property "Value" "SMTSO2540CTJ"
-			(at 218.44 99.06 0)
-			(effects
-				(font
-					(size 1.27 1.27)
-				)
-				(justify left)
-			)
-		)
-		(property "Footprint" "WA-SMSI_M2.5:Mounting_Wuerth_WA-SMSI-M2.5_H4mm_9774040151"
+			(at 218.44 96.5199 0)
+			(effects
+				(font
+					(size 1.27 1.27)
+				)
+				(justify left)
+			)
+		)
+		(property "Value" "SMTSO2040CTJ"
+			(at 218.44 99.0599 0)
+			(effects
+				(font
+					(size 1.27 1.27)
+				)
+				(justify left)
+			)
+		)
+		(property "Footprint" "Mounting_Wuerth:Mounting_Wuerth_WA-SMSI-M2_H4mm_9774040243"
 			(at 215.9 99.06 0)
 			(effects

Commit message: WIP pcb design & routing
Parts:
- removed H701, H702, H703, H704: SMTSO2040CTJ, Mounting_Wuerth:Mounting_Wuerth_WA-SMSI-M2_H4mm_9774040243, symbol Mechanical:MountingHole_Pad
- removed J701: PinHeader 1x14 P2.54mm, Connector_PinSocket_2.54mm:PinSocket_1x14_P2.54mm_Vertical, symbol Connector_Generic:Conn_01x14
- added U4: ~, display_modules:ILI9341 Module, symbol display_modules:ILI9341
Connections:
- net +3V3: now also U4.1 (VCC)
- net DC/RS: now also U4.5 (DC/RS)
- net GND: now also U4.2 (GND)
- net LED: now also U4.8 (LED)
- net MISO: now also U4.9 (MISO)
- net MOSI: now also U4.6 (MOSI)
- net SCK: now also U4.7 (SCK)
- net T_CLK: now also U4.10 (T_CLK)
- net T_CS: now also U4.11 (T_CS)
- net T_DIN: now also U4.12 (T_DIN)
- net T_DO: now also U4.13 (T_DO)
- net T_IRQ: now also U4.14 (T_IRQ)
- net ~{CS}: now also U4.3 (~{CS})
- net ~{RESET}: now also U4.4 (~{RESET})
- new net SD_MISO: U4.17 (SD_MISO)
- new net SD_MOSI: U4.16 (SD_MOSI)
- new net SD_SCK: U4.18 (SD_SCK)
- new net Touch: U4.15 (Touch)
- no-connect marks 4 -> 1
