File: pcbs/reflow-controller-v1/reflow-controller-v1.kicad_pcb (KiCad board)
At the start: 4 copper layers, 70 x 238 mm, 134 parts, among them J1 PinHeader 1x03 P2.54mm, J101 EB163A-03-C-180, J102 EB163A-02-C-180, J103 EB163A-02-C-180, J104 EB163A-02-C-180, J105 EB163A-02-C-180, J106 PinHeader 1x03 P2.54mm, J1101 EB163A-04-C-180, J1201 EB163A-04-C-180, J1301 EB163A-04-C-180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

Commit message: WIP pcb design & routing
Parts:
- removed H701, H702, H703, H704, H801, H802, H803, H804, H901, H902, H903, H904: SMTSO2040CTJ, Mounting_Wuerth:Mounting_Wuerth_WA-SMSI-M2_H4mm_9774040243
- removed J701: PinHeader 1x14 P2.54mm, Connector_PinSocket_2.54mm:PinSocket_1x14_P2.54mm_Vertical
- removed J801, J901: SSD1306 white module, Connector_PinHeader_2.54mm:PinHeader_1x04_P2.54mm_Vertical
- added C10: 100n, Capacitor_SMD:C_0603_1608Metric, B.Cu at (40.2, 72.6)
- added D1: SMAJ5.0CA, Diode_SMD:D_SMA, B.Cu at (82.2, 135.7)
- added J2: PinHeader 1x02 P2.54mm, Connector_PinHeader_2.54mm:PinHeader_1x02_P2.54mm_Vertical, B.Cu at (86.0, 134.4)
- added Q1: PMV65XP, Package_TO_SOT_SMD:SOT-23, B.Cu at (78.3, 136.1)
- added U4: ~, display_modules:ILI9341 Module, F.Cu at (53.4, 16.8)
- added U5: ~, display_modules:SSD1315 Module, F.Cu at (33.1, 119.0)
- added U6: ~, display_modules:SSD1315 Module, F.Cu at (68.5, 118.7)
- moved U1 100.7 mm to (59.9, 172.6), turned to 0 degrees
- moved D1001 65.6 mm to (39.1, 96.7)
- moved D1002 65.6 mm to (40.6, 96.7)
- moved R1001 65.6 mm to (39.1, 93.7)
- moved R1002 65.6 mm to (40.6, 93.7)
- moved BZ1 56.6 mm to (82.5, 76.1), turned to 0 degrees
- moved D201 53.3 mm to (49.2, 132.5)
- moved R205 53.3 mm to (47.6, 131.0)
- moved R201 52.6 mm to (58.7, 134.3)
- moved C203 52.6 mm to (57.4, 137.5)
- moved C204 52.6 mm to (59.8, 137.5)
- moved C205 52.6 mm to (55.3, 137.0)
- moved C207 52.6 mm to (50.6, 138.0)
- moved C208 52.6 mm to (43.8, 135.0)
- moved C209 52.6 mm to (43.8, 137.5)
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Connections:
- U1201 pad 11: /Temperature sensor 2/SDI -> /Temperature sensor 1/SDI
- U1201 pad 12: /Temperature sensor 2/SCLK -> /Temperature sensor 1/SCLK
- U1201 pad 14: /Temperature sensor 2/SDO -> /Temperature sensor 1/SDO
- U1301 pad 11: /Temperature sensor 3/SDI -> /Temperature sensor 1/SDI
- U1301 pad 12: /Temperature sensor 3/SCLK -> /Temperature sensor 1/SCLK
- U1301 pad 14: /Temperature sensor 3/SDO -> /Temperature sensor 1/SDO
- U3 pad 1: unconnected-(U3-PE2-Pad1) -> /Temperature sensor 1/SCLK
- U3 pad 10: unconnected-(U3-PF9-Pad10) -> /Temperature sensor 2/~{DRDY}
- U3 pad 11: unconnected-(U3-PF10-Pad11) -> /Temperature sensor 2/~{CS}
- U3 pad 12: unconnected-(U3-PF0-Pad12) -> /Temperature sensor 3/~{DRDY}
- U3 pad 13: unconnected-(U3-PF1-Pad13) -> /Temperature sensor 3/~{CS}
- U3 pad 15: unconnected-(U3-PC0-Pad15) -> /Servo1
- U3 pad 16: unconnected-(U3-PC1-Pad16) -> /Servo2
- U3 pad 17: unconnected-(U3-PC2-Pad17) -> /Fan_PWM
- U3 pad 26: unconnected-(U3-PA4-Pad26) -> /Buttons/LED_green
- U3 pad 27: unconnected-(U3-PA5-Pad27) -> /Buttons/LED_red
- U3 pad 3: unconnected-(U3-PE4-Pad3) -> /Buttons/Buzzer
- U3 pad 4: unconnected-(U3-PE5-Pad4) -> /Temperature sensor 1/SDO
- U3 pad 5: unconnected-(U3-PE6-Pad5) -> /Temperature sensor 1/SDI
- U3 pad 50: unconnected-(U3-PB11-Pad50) -> /Buttons/SW_2
- U3 pad 51: unconnected-(U3-PB12-Pad51) -> /Buttons/SW_Encoder
- U3 pad 52: unconnected-(U3-PB13-Pad52) -> /Display LCD/SD_SCK
- U3 pad 53: unconnected-(U3-PB14-Pad53) -> /Display LCD/SD_MISO
- U3 pad 54: unconnected-(U3-PB15-Pad54) -> /Display LCD/SD_MOSI
- U3 pad 55: unconnected-(U3-PD8-Pad55) -> /Display LCD/Touch
- U3 pad 56: unconnected-(U3-PD9-Pad56) -> /Buttons/SW_1
- U3 pad 57: unconnected-(U3-PD10-Pad57) -> /SSR 2/IN
- U3 pad 58: unconnected-(U3-PD11-Pad58) -> /SSR 4/IN
- U3 pad 59: unconnected-(U3-PD12-Pad59) -> /Buttons/Encoder_A
- U3 pad 60: unconnected-(U3-PD13-Pad60) -> /Buttons/Encoder_B
- U3 pad 61: unconnected-(U3-PD14-Pad61) -> /SSR 1/IN
- U3 pad 62: unconnected-(U3-PD15-Pad62) -> /SSR 3/IN
- U3 pad 65: unconnected-(U3-PC6-Pad65) -> /Display OLED 2/I2C_SCL
- U3 pad 66: unconnected-(U3-PC7-Pad66) -> /Display OLED 2/I2C_SDA
- U3 pad 67: unconnected-(U3-PC8-Pad67) -> /Display OLED 1/I2C_SCL
- U3 pad 68: unconnected-(U3-PC9-Pad68) -> /Display OLED 1/I2C_SDA
- U3 pad 69: unconnected-(U3-PA8-Pad69) -> /Temperature onboard 1/SDA
- U3 pad 70: unconnected-(U3-PA9-Pad70) -> /Temperature onboard 1/SCL
- U3 pad 78: unconnected-(U3-PA15-Pad78) -> /Display LCD/T_IRQ
- U3 pad 79: unconnected-(U3-PC10-Pad79) -> /Display LCD/T_CLK
- U3 pad 8: unconnected-(U3-PC14-Pad8) -> /Temperature sensor 1/~{DRDY}
- U3 pad 80: unconnected-(U3-PC11-Pad80) -> /Display LCD/T_DO
- U3 pad 81: unconnected-(U3-PC12-Pad81) -> /Display LCD/T_DIN
- U3 pad 82: unconnected-(U3-PD0-Pad82) -> /Display LCD/T_CS
- U3 pad 89: unconnected-(U3-PD7-Pad89) -> /Display LCD/LED
- U3 pad 9: unconnected-(U3-PC15-Pad9) -> /Temperature sensor 1/~{CS}
- U3 pad 90: unconnected-(U3-PB3-Pad90) -> /Display LCD/SCK
- U3 pad 91: unconnected-(U3-PB4-Pad91) -> /Display LCD/MISO
- U3 pad 92: unconnected-(U3-PB5-Pad92) -> /Display LCD/MOSI
- U3 pad 93: unconnected-(U3-PB6-Pad93) -> /Display LCD/DC/RS
- U3 pad 94: unconnected-(U3-PB7-Pad94) -> /Display LCD/~{RESET}
- U3 pad 97: unconnected-(U3-PE0-Pad97) -> /Display LCD/~{CS}
Routing:
- net /Temperature onboard 1/SCL: track 0.00 -> 144.4 mm, vias 0 -> 2
- net /Temperature onboard 1/SDA: track 0.00 -> 140.0 mm, vias 0 -> 2
- net /Buttons/SW_2: track 0.00 -> 130.3 mm, vias 0 -> 1
- net /SSR 2/IN: track 0.00 -> 116.5 mm
- net /SSR 4/IN: track 0.00 -> 110.5 mm
- net /Buttons/SW_Encoder: track 0.00 -> 110.0 mm
- net /SSR 1/IN: track 0.00 -> 103.5 mm
- net /SSR 3/IN: track 0.00 -> 100.9 mm
- net /Buttons/SW_1: track 0.00 -> 92.0 mm, vias 0 -> 1
- net /Buttons/Encoder_A: track 0.00 -> 90.3 mm, vias 0 -> 2
- net /Buttons/Encoder_B: track 0.00 -> 85.8 mm, vias 0 -> 2
- net +5V: track 23.9 -> 102.7 mm
- net /Display LCD/~{CS}: track 0.00 -> 72.0 mm
- net /Display LCD/~{RESET}: track 0.00 -> 70.4 mm
- net /Display LCD/DC/RS: track 0.00 -> 68.4 mm
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Other:
- board text added: "- SPI Display - Spi touch - SPI temp - spi sd card - I2C temp onboad - I2C oled1 - I2C oled2"
- board text added: "TODO: - Find fitting mounting for display - Connect earth to Digital ground? - Correct display mounting - correct pcb dimensions - pcb mounting"

Commit message: update routing with new mechanical positioning
Parts:
- added H1: MountingHole_Pad, Mounting_Wuerth:Mounting_Wuerth_WA-SMSI-M3_H15mm_9774150360, B.Cu at (31.1, 19.2)
- added H2: MountingHole_Pad, Mounting_Wuerth:Mounting_Wuerth_WA-SMSI-M3_H15mm_9774150360, B.Cu at (97.6, 26.2)
- added H3: MountingHole_Pad, Mounting_Wuerth:Mounting_Wuerth_WA-SMSI-M3_H15mm_9774150360, B.Cu at (97.6, 66.2)
- added H4: MountingHole_Pad, Mounting_Wuerth:Mounting_Wuerth_WA-SMSI-M3_H15mm_9774150360, B.Cu at (34.6, 131.2)
- added H5: MountingHole_Pad, Mounting_Wuerth:Mounting_Wuerth_WA-SMSI-M3_H15mm_9774150360, B.Cu at (52.6, 131.2)
- added H6: MountingHole_Pad, Mounting_Wuerth:Mounting_Wuerth_WA-SMSI-M3_H15mm_9774150360, B.Cu at (76.6, 131.2)
- added H7: MountingHole_Pad, Mounting_Wuerth:Mounting_Wuerth_WA-SMSI-M3_H15mm_9774150360, B.Cu at (97.6, 131.2)
- added H8: MountingHole_Pad, Mounting_Wuerth:Mounting_Wuerth_WA-SMSI-M3_H15mm_9774150360, B.Cu at (97.6, 236.2)
- added H9: MountingHole_Pad, Mounting_Wuerth:Mounting_Wuerth_WA-SMSI-M3_H15mm_9774150360, B.Cu at (23.1, 244.2)
- U2: moved to B.Cu
- moved U1 105.6 mm to (21.1, 74.4), turned to 180 degrees
- moved C301 83.1 mm to (45.7, 149.4), turned to 0 degrees
- moved R305 79.2 mm to (37.7, 151.3), turned to 0 degrees
- moved J102 78.4 mm to (60.3, 159.3), turned to 180 degrees
- moved C211 69.0 mm to (69.9, 78.5), turned to 90 degrees
- moved L201 68.3 mm to (80.8, 81.3), turned to 180 degrees
- moved C210 67.7 mm to (72.2, 78.5), turned to 90 degrees
- moved C207 67.5 mm to (84.4, 79.6), turned to 90 degrees
- moved C206 66.8 mm to (85.9, 79.6), turned to 90 degrees
- moved C209 66.5 mm to (74.5, 78.5), turned to 90 degrees
- moved R206 66.0 mm to (88.1, 80.8), turned to -90 degrees
- moved C208 65.4 mm to (76.9, 78.5), turned to 90 degrees
- moved D301 63.4 mm to (39.9, 159.1), turned to 180 degrees
- moved U201 62.3 mm to (85.5, 82.8), turned to 90 degrees
- moved R204 61.7 mm to (88.8, 83.1), turned to 0 degrees
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Connections:
- U3 pad 57: /SSR 2/IN -> /SSR 1/IN
- U3 pad 58: /SSR 4/IN -> /SSR 2/IN
- U3 pad 61: /SSR 1/IN -> /SSR 3/IN
- U3 pad 62: /SSR 3/IN -> /SSR 4/IN
Routing:
- net /Temperature sensor 3/~{CS}: track 0.00 -> 52.1 mm
- net /Temperature sensor 3/~{DRDY}: track 0.00 -> 46.3 mm
- net Net-(R302-Pad1): track 47.4 -> 2.51 mm
- net /SSR 4/IN: track 110.5 -> 148.3 mm
- net /Phase_N: track 174.5 -> 136.8 mm, vias 7 -> 0
- net /Temperature sensor 2/~{CS}: track 0.00 -> 37.1 mm
- net /Temperature onboard 1/SCL: track 144.4 -> 110.4 mm
- net Net-(R403-Pad1): track 36.4 -> 2.51 mm, vias 2 -> 0
- net /Buttons/SW_2: track 130.3 -> 97.9 mm
- net /Temperature sensor 2/~{DRDY}: track 0.00 -> 31.2 mm
- net +5V: track 102.7 -> 133.3 mm, vias 0 -> 3
- net /Buttons/SW_Encoder: track 110.0 -> 79.5 mm
- net /Temperature onboard 1/SDA: track 140.0 -> 110.6 mm, vias 2 -> 3
- net /Temperature sensor 1/~{CS}: track 0.00 -> 28.5 mm, vias 0 -> 2
- net /SSR 3/IN: track 100.9 -> 128.3 mm
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- added copper zone on B.Cu, net +3V3
- added copper zone on In2.Cu, net +3V3
- added copper zone on B.Cu, net +5V
- added copper zone on B.Cu, net /Prefuse_L
- added copper zone on B.Cu, net /Prefuse_N
- added copper zone on B.Cu, net /SSR 1/MAIN_OUT
- added copper zone on B.Cu, net /SSR 2/MAIN_OUT
- added copper zone on B.Cu, net /SSR 3/MAIN_OUT
- added copper zone on B.Cu, net /SSR 4/MAIN_OUT
- added copper zone on In1.Cu, net GND
- removed copper zone on In1.Cu, net +3V3
Other:
- board size 70 x 238 mm -> 85.2 x 238.5 mm
- board text added: "N|E|L"
- board text added: "TODO: - Find fitting mounting for display - Connect earth to Digital ground? - Correct display mounting"
- board text removed: "L|E|N"
- board text removed: "TODO: - Find fitting mounting for display - Connect earth to Digital ground? - Correct display mounting - correct pcb dimensions - pcb mounting"

Commit message: increase isolation distance
Parts:
- moved C401 9.78 mm to (36.7, 177.6)
- moved D601 9.78 mm to (35.8, 225.6)
- moved R402 9.78 mm to (43.7, 194.0)
- moved R403 9.78 mm to (28.8, 194.0)
- moved R501 9.78 mm to (20.5, 212.8)
- moved U601 9.78 mm to (23.5, 227.1)
- moved R504 9.78 mm to (30.9, 198.4)
- moved C301 9.78 mm to (41.5, 158.2)
- moved C501 9.78 mm to (36.7, 196.8)
- moved C601 9.78 mm to (36.7, 216.0)
- moved D301 9.78 mm to (35.8, 168.0)
- moved D401 9.78 mm to (35.8, 187.2)
- moved D501 9.78 mm to (35.8, 206.4)
- moved J102 9.78 mm to (56.2, 168.2)
- moved J103 9.78 mm to (56.2, 182.7)
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Routing:
- net /SSR 2/IN: track 106.8 -> 116.4 mm
- net GND: track 69.4 -> 78.9 mm, vias 45 -> 57
- net /SSR 4/IN: track 148.3 -> 157.5 mm
- net /SSR 1/IN: track 86.6 -> 95.7 mm
- net /SSR 3/IN: track 128.3 -> 137.3 mm
- net Earth_Protective: track 0.00 -> 8.20 mm
- net +5V: track 133.3 -> 140.6 mm
- net +3V3: track 106.3 -> 109.4 mm, vias 28 -> 29
- net /Temperature onboard 1/SDA: track 110.6 -> 113.1 mm
- net /Temperature onboard 1/SCL: track 110.4 -> 112.8 mm
- net /Phase_L: track 160.3 -> 162.5 mm, vias 37 -> 45
- net /Phase_N: track 136.8 -> 135.7 mm

Commit message: add debug uart & swd
Parts:
- added J3: SWD, Connector_Molex:Molex_KK-254_AE-6410-03A_1x03_P2.54mm_Vertical, B.Cu at (29.5, 60.8)
- added J4: UART, Connector_Molex:Molex_KK-254_AE-6410-03A_1x03_P2.54mm_Vertical, B.Cu at (29.5, 56.6)
Connections:
- U3 pad 30: unconnected-(U3-PC4-Pad30) -> Net-(J4-Pin_3)
- U3 pad 31: unconnected-(U3-PC5-Pad31) -> Net-(J4-Pin_2)
- U3 pad 76: unconnected-(U3-PA13-Pad76) -> Net-(J3-Pin_3)
- U3 pad 77: unconnected-(U3-PA14-Pad77) -> Net-(J3-Pin_1)
Routing:
- net Net-(J4-Pin_3): track 0.00 -> 41.3 mm, vias 0 -> 1
- net Net-(J4-Pin_2): track 0.00 -> 38.0 mm, vias 0 -> 1
- net Net-(J3-Pin_1): track 0.00 -> 10.6 mm
- net Net-(J3-Pin_3): track 0.00 -> 5.30 mm
Other:
- board text added: "TODO: - Find fitting mounting for display - Connect earth to Digital ground? - Correct display mounting - Ground/eath mounting holes? - Plane/Via Stitching"
- board text removed: "TODO: - Find fitting mounting for display - Connect earth to Digital ground? - Correct display mounting"

Commit message: update debug power footprint
Parts:
- J2: footprint Connector_PinHeader_2.54mm:PinHeader_1x02_P2.54mm_Vertical -> Connector_Molex:Molex_KK-254_AE-6410-02A_1x02_P2.54mm_Vertical
- moved J2 1.67 mm to (69.2, 99.2), turned to 90 degrees
Routing:
- net Net-(D1-A2): track 7.47 -> 9.20 mm
- net GND: track 78.9 -> 80.5 mm
Changed lines of the file:
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@@
 		)
 	)
-	(footprint "Connector_PinHeader_2.54mm:PinHeader_1x02_P2.54mm_Vertical"
+	(footprint "Connector_Molex:Molex_KK-254_AE-6410-02A_1x02_P2.54mm_Vertical"
 		(layer "B.Cu")
-		(at 70.8717 99.3648)
-		(descr "Through hole straight pin header, 1x02, 2.54mm pitch, single row")
-		(tags "Through hole pin header THT 1x02 2.54mm single row")
+		(at 69.215 99.187 90)
+		(descr "Molex KK-254 Interconnect System, old/engineering part number: AE-6410-02A example for new part number: 22-27-2021, 2 Pins (http://www.molex.com/pdm_docs/sd/022272021_sd.pdf), generated with kicad-footprint-generator")
+		(tags "connector Molex KK-254 vertical")
 		(property "Reference" "J2"
-			(at 0 2.33 0)
+			(at 1.27 4.12 90)
 			(layer "B.SilkS")
 			(effects
@@
 		)
 		(property "Value" "PinHeader 1x02 P2.54mm"
-			(at 0 -4.87 0)
+			(at 1.27 -4.08 90)
 			(layer "B.Fab")
 			(effects
@@
 			)
 		)
-		(property "Footprint" "Connector_PinHeader_2.54mm:PinHeader_1x02_P2.54mm_Vertical"
-			(at 0 0 180)
+		(property "Footprint" "Connector_Molex:Molex_KK-254_AE-6410-02A_1x02_P2.54mm_Vertical"
+			(at 0 0 -90)
 			(unlocked yes)
 			(layer "B.Fab")
@@
 		)
 		(property "Datasheet" ""
-			(at 0 0 180)
+			(at 0 0 -90)
 			(unlocked yes)
 			(layer "B.Fab")
@@
 		)
 		(property "Description" "Generic connector, single row, 01x02, script generated (kicad-library-utils/schlib/autogen/connector/)"
-			(at 0 0 180)
+			(at 0 0 -90)
 			(unlocked yes)
 			(layer "B.Fab")
@@
 		(attr through_hole)
 		(fp_line
-			(start -1.33 -3.87)
-			(end -1.33 -1.27)
+			(start 3.92 -2.99)
+			(end -1.38 -2.99)
 			(stroke
 				(width 0.12)
@@
 		)
 		(fp_line
-			(start -1.33 1.33)
-			(end -1.33 0)
+			(start 2.54 -2.99)
+			(end 2.54 -1.99)
 			(stroke
 				(width 0.12)
@@
 		)
 		(fp_line
-			(start 0 1.33)
-			(end -1.33 1.33)
+			(start -1.38 -2.99)
+			(end -1.38 3.03)
 			(stroke
 				(width 0.12)
@@
 		)
 		(fp_line
-			(start 1.33 -3.87)
-			(end -1.33 -3.87)
+			(start -1.67 -2)
+			(end -1.67 2)
 			(stroke
 				(width 0.12)
@@
 		)
 		(fp_line
-			(start 1.33 -3.87)
-			(end 1.33 -1.27)
+			(start 2.54 -1.99)
+			(end 0 -1.99)
 			(stroke
 				(width 0.12)
@@
 		)
 		(fp_line
-			(start 1.33 -1.27)
-			(end -1.33 -1.27)
+			(start 2.54 -1.99)
+			(end 2.29 -1.46)
 			(stroke
 				(width 0.12)
@@
 		)
 		(fp_line
-			(start -1.8 -4.35)
-			(end -1.8 1.8)
+			(start 2.29 -1.99)
+			(end 2.29 -2.99)
+			(stroke
+				(width 0.12)
+				(type solid)
+			)
+			(layer "B.SilkS")
+		)
+		(fp_line
+			(start 0.25 -1.99)
+			(end 0.25 -2.99)
+			(stroke
+				(width 0.12)
+				(type solid)
+			)
+			(layer "B.SilkS")
+		)
+		(fp_line
+			(start 0 -1.99)
+			(end 0 -2.99)
+			(stroke
+				(width 0.12)
+				(type solid)
+			)
+			(layer "B.SilkS")
+		)
+		(fp_line
+			(start 2.29 -1.46)
+			(end 0.25 -1.46)
+			(stroke
+				(width 0.12)
+				(type solid)
+			)
+			(layer "B.SilkS")
+		)
+		(fp_line
+			(start 0.25 -1.46)
+			(end 0 -1.99)
+			(stroke
+				(width 0.12)
+				(type solid)
+			)
+			(layer "B.SilkS")
+		)
+		(fp_line
+			(start 3.34 2.43)
+			(end 1.74 2.43)
+			(stroke
+				(width 0.12)
+				(type solid)
+			)
+			(layer "B.SilkS")
+		)
+		(fp_line
+			(start 1.74 2.43)
+			(end 1.74 3.03)
+			(stroke
+				(width 0.12)
+				(type solid)
+			)
+			(layer "B.SilkS")
+		)
+		(fp_line
+			(start 0.8 2.43)
+			(end -0.8 2.43)
+			(stroke
+				(width 0.12)
+				(type solid)
+			)
+			(layer "B.SilkS")
+		)
+		(fp_line
+			(start -0.8 2.43)
+			(end -0.8 3.03)
+			(stroke
+				(width 0.12)
+				(type solid)
+			)
+			(layer "B.SilkS")
+		)
+		(fp_line
+			(start 3.92 3.03)
+			(end 3.92 -2.99)
+			(stroke
+				(width 0.12)
+				(type solid)
+			)
+			(layer "B.SilkS")
+		)
+		(fp_line
+			(start 3.34 3.03)
+			(end 3.34 2.43)
+			(stroke
+				(width 0.12)
+				(type solid)
+			)
+			(layer "B.SilkS")
+		)
+		(fp_line
+			(start 0.8 3.03)
+			(end 0.8 2.43)
+			(stroke
+				(width 0.12)
+				(type solid)
+			)
+			(layer "B.SilkS")
+		)
+		(fp_line
+			(start -1.38 3.03)
+			(end 3.92 3.03)
+			(stroke
+				(width 0.12)
+				(type solid)
+			)
+			(layer "B.SilkS")
+		)
+		(fp_line
+			(start 4.31 -3.38)
+			(end -1.77 -3.38)
 			(stroke
 				(width 0.05)
@@
 		)
 		(fp_line
-			(start -1.8 1.8)
-			(end 1.8 1.8)
+			(start -1.77 -3.38)
+			(end -1.77 3.42)
 			(stroke
 				(width 0.05)
@@
 		)
 		(fp_line
-			(start 1.8 -4.35)
-			(end -1.8 -4.35)
+			(start 4.31 3.42)
+			(end 4.31 -3.38)
 			(stroke
 				(width 0.05)
@@
 		)
 		(fp_line
-			(start 1.8 1.8)
-			(end 1.8 -4.35)
+			(start -1.77 3.42)
+			(end 4.31 3.42)
 			(stroke
 				(width 0.05)
@@
 		)
 		(fp_line
-			(start -1.27 -3.81)
-			(end 1.27 -3.81)
+			(start 3.81 -2.88)
+			(end -1.27 -2.88)
 			(stroke
 				(width 0.1)
@@
 		)
 		(fp_line
-			(start -1.27 0.635)
-			(end -1.27 -3.81)
+			(start -1.27 -2.88)
+			(end -1.27 2.92)
 			(stroke
 				(width 0.1)
@@
 		)
 		(fp_line
-			(start -0.635 1.27)
-			(end -1.27 0.635)
+			(start -1.27 -0.5)
+			(end -0.562893 0)
 			(stroke
 				(width 0.1)
@@
 		)
 		(fp_line
-			(start 1.27 -3.81)
-			(end 1.27 1.27)
+			(start -0.562893 0)
+			(end -1.27 0.5)
 			(stroke
 				(width 0.1)
@@
 		)
 		(fp_line
-			(start 1.27 1.27)
-			(end -0.635 1.27)
+			(start 3.81 2.92)
+			(end 3.81 -2.88)
+			(stroke
+				(width 0.1)
+				(type solid)
+			)
+			(layer "B.Fab")
+		)
+		(fp_line
+			(start -1.27 2.92)
+			(end 3.81 2.92)
 			(stroke
 				(width 0.1)
@@
 		)
 		(fp_text user "${REFERENCE}"
-			(at 0 -1.27 90)
+			(at 1.27 2.22 90)
 			(layer "B.Fab")
 			(effects
@@
 			)
 		)
-		(pad "1" thru_hole rect
-			(at 0 0)
-			(size 1.7 1.7)
-			(drill 1)
+		(pad "1" thru_hole roundrect
+			(at 0 0 90)
+			(size 1.74 2.19)
+			(drill 1.19)
 			(layers "*.Cu" "*.Mask")
 			(remove_unused_layers no)
+			(roundrect_rratio 0.143678)
 			(net 177 "Net-(D1-A2)")
 			(pinfunction "Pin_1")
@@
 		)
 		(pad "2" thru_hole oval
-			(at 0 -2.54)
-			(size 1.7 1.7)
-			(drill 1)
+			(at 2.54 0 90)
+			(size 1.74 2.19)
+			(drill 1.19)
 			(layers "*.Cu" "*.Mask")
 			(remove_unused_layers no)
@@
 			(pintype "passive")
 		)
-		(model "${KICAD8_3DMODEL_DIR}/Connector_PinHeader_2.54mm.3dshapes/PinHeader_1x02_P2.54mm_Vertical.wrl"
+		(model "${KICAD8_3DMODEL_DIR}/Connector_Molex.3dshapes/Molex_KK-254_AE-6410-02A_1x02_P2.54mm_Vertical.wrl"
 			(offset
 				(xyz 0 0 0)
@@
 	)
 	(segment
-		(start 71.5509 96.1456)
-		(end 70.8717 96.8248)
-		(width 0.5)
+		(start 20.1574 74.672)
+		(end 20.1574 75.172)
+		(width 0.2)
 		(layer "B.Cu")
 		(net 1)
 	)
 	(segment
-		(start 20.1574 74.672)
-		(end 20.1574 75.172)
-		(width 0.2)
+		(start 69.7164 96.1456)
+		(end 69.215 96.647)
+		(width 0.5)
 		(layer "B.Cu")
 		(net 1)
@@
 	)
 	(segment
-		(start 74.4277 96.1456)
-		(end 71.5509 96.1456)
-		(width 0.5)
-		(layer "B.Cu")
-		(net 1)
-	)
-	(segment
 		(start 57.646 147.7638)
 		(end 60.5536 144.8562)
@@
 	)
 	(segment
+		(start 74.4277 96.1456)
+		(end 69.7164 96.1456)
+		(width 0.5)
+		(layer "B.Cu")
+		(net 1)
+	)
+	(segment
 		(start 37.485 87.059)
 		(end 37.485 87.953)
@@
 	)
 	(segment
-		(start 70.8717 99.3648)
-		(end 73.6469 99.3648)
+		(start 69.215 99.187)
+		(end 73.4691 99.187)
 		(width 0.5)
 		(layer "B.Cu")
@@
 	)
 	(segment
-		(start 76.4633 98.11)
+		(start 73.4691 99.187)
 		(end 74.4277 100.1456)
 		(width 0.5)
@@
 	)
 	(segment
-		(start 73.6469 99.3648)
+		(start 76.4633 98.11)
 		(end 74.4277 100.1456)
 		(width 0.5)

Commit message: label uart & swd
Connections:
- net Net-(J3-Pin_1) renamed /microcontroller/SWCLK
- net Net-(J3-Pin_3) renamed /microcontroller/SWDIO
- net Net-(J4-Pin_2) renamed /microcontroller/USART1_RX
- net Net-(J4-Pin_3) renamed /microcontroller/USART1_TX
Changed lines of the file:
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@@
 	(net 112 "unconnected-(U3-PD3-Pad85)")
 	(net 113 "unconnected-(U3-PA10-Pad71)")
-	(net 114 "Net-(J3-Pin_3)")
+	(net 114 "/microcontroller/SWDIO")
 	(net 115 "unconnected-(U3-PE15-Pad46)")
 	(net 116 "unconnected-(U3-PE11-Pad42)")
@@
 	(net 129 "unconnected-(U3-PD6-Pad88)")
 	(net 130 "unconnected-(U3-PE7-Pad38)")
-	(net 131 "Net-(J3-Pin_1)")
-	(net 132 "Net-(J4-Pin_2)")
-	(net 133 "Net-(J4-Pin_3)")
+	(net 131 "/microcontroller/SWCLK")
+	(net 132 "/microcontroller/USART1_RX")
+	(net 133 "/microcontroller/USART1_TX")
 	(net 134 "unconnected-(U301-NC-Pad3)")
 	(net 135 "unconnected-(U301-NC-Pad5)")
@@
 			(remove_unused_layers no)
 			(roundrect_rratio 0.143678)
-			(net 131 "Net-(J3-Pin_1)")
+			(net 131 "/microcontroller/SWCLK")
 			(pinfunction "Pin_1")
 			(pintype "passive")
@@
 			(layers "*.Cu" "*.Mask")
 			(remove_unused_layers no)
-			(net 114 "Net-(J3-Pin_3)")
+			(net 114 "/microcontroller/SWDIO")
 			(pinfunction "Pin_3")
 			(pintype "passive")
@@
 			(layers "*.Cu" "*.Mask")
 			(remove_unused_layers no)
-			(net 132 "Net-(J4-Pin_2)")
+			(net 132 "/microcontroller/USART1_RX")
 			(pinfunction "Pin_2")
 			(pintype "passive")
@@
 			(layers "*.Cu" "*.Mask")
 			(remove_unused_layers no)
-			(net 133 "Net-(J4-Pin_3)")
+			(net 133 "/microcontroller/USART1_TX")
 			(pinfunction "Pin_3")
 			(pintype "passive")
@@
 			(layers "B.Cu" "B.Paste" "B.Mask")
 			(roundrect_rratio 0.25)
-			(net 133 "Net-(J4-Pin_3)")
+			(net 133 "/microcontroller/USART1_TX")
 			(pinfunction "PC4")
 			(pintype "bidirectional")
@@
 			(layers "B.Cu" "B.Paste" "B.Mask")
 			(roundrect_rratio 0.25)
-			(net 132 "Net-(J4-Pin_2)")
+			(net 132 "/microcontroller/USART1_RX")
 			(pinfunction "PC5")
 			(pintype "bidirectional")
@@
 			(layers "B.Cu" "B.Paste" "B.Mask")
 			(roundrect_rratio 0.25)
-			(net 114 "Net-(J3-Pin_3)")
+			(net 114 "/microcontroller/SWDIO")
 			(pinfunction "PA13")
 			(pintype "bidirectional")
@@
 			(layers "B.Cu" "B.Paste" "B.Mask")
 			(roundrect_rratio 0.25)
-			(net 131 "Net-(J3-Pin_1)")
+			(net 131 "/microcontroller/SWCLK")
 			(pinfunction "PA14")
 			(pintype "bidirectional")
