File: pcbs/reflow-controller-v1/reflow-controller-v1.kicad_pcb (KiCad board)
At the start: 4 copper layers, 74.9 x 243.5 mm, 149 parts, among them J1 PinHeader 1x03 P2.54mm, J101 EB163A-03-C-180, J102 EB163A-02-C-180, J103 EB163A-02-C-180, J104 EB163A-02-C-180, J105 EB163A-02-C-180, J106 PinHeader 1x03 P2.54mm, J1101 EB163A-04-C-180, J1201 EB163A-04-C-180, J1301 EB163A-04-C-180, J201 PinHeader 1x02 P2.54mm, J3 SWD, J4 UART, M101 47053-1000, Q1601 MMBT3904, Q1602 140357145200, Q201 PMV65XP, SW1001 TS04-66-85-BK-160-SMT, SW1002 PEC12R-3220F-S0024, SW1003 TS04-66-85-BK-160-SMT, U1 TMP1075DSG, U1101 MAX31865ATP+, U1201 MAX31865ATP+, U1301 MAX31865ATP+, U201 TPS62933DRLR, U202 AZ1117-3.3, U3 STM32G474VETx, U301 MOC3043SM, U401 MOC3043SM, U501 MOC3043SM, U601 MOC3043SM

Commit message: pcb routing touchups
Parts:
- moved J3 5.79 mm to (35.6, 84.2)
- moved BZ1 2.41 mm to (32.5, 95.8)
- moved R5 2.20 mm to (38.5, 95.4)
Routing:
- net /microcontroller/SWDIO: track 8.47 -> 14.3 mm
- net /microcontroller/SWCLK: track 7.85 -> 13.6 mm
- net /Buttons/Buzzer: track 15.3 -> 16.8 mm
- net Net-(BZ1-+): track 2.30 -> 1.80 mm
Other:
- board text removed: "- SPI Display - Spi touch - SPI temp - spi sd card - I2C temp onboad - I2C oled1 - I2C oled2"
Changed lines of the file:
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@@
 	(footprint "Resistor_SMD:R_0603_1608Metric"
 		(layer "B.Cu")
-		(at 39.1692 93.296 -90)
+		(at 38.458 95.3788 -90)
 		(descr "Resistor SMD 0603 (1608 Metric), square (rectangular) end terminal, IPC_7351 nominal, (Body size source: IPC-SM-782 page 72, https://www.pcb-3d.com/wordpress/wp-content/uploads/ipc-sm-782a_amendment_1_and_2.pdf), generated with kicad-footprint-generator")
 		(tags "resistor")
@@
 	(footprint "Connector_Molex:Molex_KK-254_AE-6410-03A_1x03_P2.54mm_Vertical"
 		(layer "B.Cu")
-		(at 41.4044 84.2028 -90)
+		(at 35.6132 84.2028 -90)
 		(descr "Molex KK-254 Interconnect System, old/engineering part number: AE-6410-03A example for new part number: 22-27-2031, 3 Pins (http://www.molex.com/pdm_docs/sd/022272021_sd.pdf), generated with kicad-footprint-generator")
 		(tags "connector Molex KK-254 vertical")
@@
 	(footprint "Buzzer_Beeper:Buzzer_Murata_PKMCS0909E"
 		(layer "B.Cu")
-		(at 32.792 93.4508 180)
+		(at 32.4636 95.836 180)
 		(descr "Murata Buzzer http://www.murata.com/en-us/api/pdfdownloadapi?cate=&partno=PKMCS0909E4000-R1")
 		(tags "Murata Buzzer Beeper")
@@
 		)
 	)
-	(gr_text "- SPI Display\n- Spi touch\n- SPI temp\n- spi sd card\n- I2C temp onboad\n- I2C oled1\n- I2C oled2"
-		(at 155.6258 94.996 0)
-		(layer "Cmts.User")
-		(effects
-			(font
-				(size 1.5 1.5)
-				(thickness 0.1875)
-			)
-			(justify left bottom)
-		)
-	)
 	(gr_text "Standofs NEED to be at least 23mm to clear the DCDC module"
 		(at 119.484 107.012 0)
@@
 	)
 	(gr_text "TODO:\n- Plane/Via Stitching"
-		(at 153.2382 62.4586 0)
+		(at 122.3796 56.3136 0)
 		(layer "Cmts.User")
 		(effects
@@
 	)
 	(segment
-		(start 57.5588 93.819046)
-		(end 58.1888 93.189046)
+		(start 58.283 145.5692)
+		(end 57.5588 144.845)
 		(width 0.2)
 		(layer "F.Cu")
@@
 	)
 	(segment
-		(start 57.5588 143.123914)
-		(end 57.5588 93.819046)
+		(start 57.5588 93.819046)
+		(end 58.1888 93.189046)
 		(width 0.2)
 		(layer "F.Cu")
@@
 	)
 	(segment
-		(start 58.248043 143.813157)
-		(end 57.5588 143.123914)
+		(start 57.5588 144.845)
+		(end 57.5588 93.819046)
 		(width 0.2)
 		(layer "F.Cu")
@@
 	)
 	(via
-		(at 58.248043 143.813157)
+		(at 58.283 145.5692)
 		(size 0.6)
 		(drill 0.3)
@@
 	)
 	(segment
-		(start 58.283 149.0752)
+		(start 58.283 145.5692)
 		(end 58.283 146.636)
 		(width 0.2)
@@
 	)
 	(segment
-		(start 58.8918 149.684)
-		(end 58.283 149.0752)
-		(width 0.2)
-		(layer "B.Cu")
-		(net 10)
-	)
-	(segment
-		(start 58.248043 143.813157)
-		(end 58.283 143.848114)
+		(start 58.283 149.0752)
+		(end 58.283 146.636)
 		(width 0.2)
 		(layer "B.Cu")
@@
 	)
 	(segment
-		(start 58.283 143.848114)
-		(end 58.283 146.636)
+		(start 58.8918 149.684)
+		(end 58.283 149.0752)
 		(width 0.2)
 		(layer "B.Cu")
@@
 	)
 	(segment
-		(start 39.1692 94.121)
-		(end 37.8122 94.121)
+		(start 38.458 96.2038)
+		(end 37.1814 96.2038)
 		(width 0.2)
 		(layer "B.Cu")
@@
 	)
 	(segment
-		(start 37.8122 94.121)
-		(end 37.142 93.4508)
+		(start 37.1814 96.2038)
+		(end 36.8136 95.836)
 		(width 0.2)
 		(layer "B.Cu")
@@
 	)
 	(segment
+		(start 55.9588 142.2768)
+		(end 55.9588 141.779744)
+		(width 0.2)
+		(layer "F.Cu")
+		(net 58)
+	)
+	(segment
 		(start 53.471643 104.98)
-		(end 56.3588 107.867157)
+		(end 53.1888 104.98)
 		(width 0.2)
 		(layer "F.Cu")
@@
 	)
 	(segment
-		(start 53.1888 104.98)
-		(end 53.471643 104.98)
+		(start 55.9588 141.779744)
+		(end 56.3588 141.379744)
+		(width 0.2)
+		(layer "F.Cu")
+		(net 58)
+	)
+	(segment
+		(start 56.3588 141.379744)
+		(end 56.3588 107.867157)
 		(width 0.2)
 		(layer "F.Cu")
@@
 	(segment
 		(start 56.3588 107.867157)
-		(end 56.3588 138.118527)
+		(end 53.471643 104.98)
 		(width 0.2)
 		(layer "F.Cu")
@@
 	)
 	(segment
-		(start 56.3588 138.118527)
-		(end 55.954548 138.522779)
+		(start 56.5588 142.8768)
+		(end 55.9588 142.2768)
 		(width 0.2)
 		(layer "F.Cu")
@@
 	)
 	(via
-		(at 55.954548 138.522779)
+		(at 56.5588 142.8768)
 		(size 0.6)
 		(drill 0.3)
@@
 	)
 	(segment
-		(start 55.954548 138.522779)
-		(end 55.954548 139.291348)
+		(start 60.5052 146.7376)
+		(end 60.5052 154.6116)
 		(width 0.2)
 		(layer "B.Cu")
@@
 	)
 	(segment
-		(start 55.954548 139.291348)
-		(end 60.5052 143.842)
+		(start 60.06 155.0568)
+		(end 60.5052 154.6116)
 		(width 0.2)
 		(layer "B.Cu")
@@
 	)
 	(segment
-		(start 60.06 155.0568)
-		(end 60.5052 154.6116)
+		(start 56.5588 142.8768)
+		(end 56.6444 142.8768)
 		(width 0.2)
 		(layer "B.Cu")
@@
 	)
 	(segment
-		(start 53.2888 88.74781)
-		(end 53.1888 88.84781)
+		(start 56.6444 142.8768)
+		(end 60.5052 146.7376)
 		(width 0.2)
 		(layer "B.Cu")
@@
 	)
 	(segment
-		(start 60.5052 143.842)
-		(end 60.5052 154.6116)
+		(start 53.2888 88.74781)
+		(end 53.1888 88.84781)
 		(width 0.2)
 		(layer "B.Cu")
@@
 	)
 	(segment
-		(start 56.7588 107.701471)
-		(end 52.640329 103.583)
+		(start 52.640329 103.583)
+		(end 52.5888 103.583)
 		(width 0.2)
 		(layer "F.Cu")
@@
 	)
 	(segment
-		(start 56.7588 138.847072)
+		(start 56.7588 141.828273)
 		(end 56.7588 107.701471)
 		(width 0.2)
@@
 	)
 	(segment
-		(start 52.640329 103.583)
-		(end 52.5888 103.583)
+		(start 56.7588 107.701471)
+		(end 52.640329 103.583)
 		(width 0.2)
 		(layer "F.Cu")
@@
 	)
 	(segment
-		(start 56.5588 139.047072)
-		(end 56.7588 138.847072)
+		(start 56.5588 142.028273)
+		(end 56.7588 141.828273)
 		(width 0.2)
 		(layer "F.Cu")
@@
 	)
 	(via
-		(at 56.5588 139.047072)
+		(at 56.5588 142.028273)
 		(size 0.6)
 		(drill 0.3)
@@
 	)
 	(segment
-		(start 59.924443 142.695557)
-		(end 59.924443 142.695558)
-		(width 0.2)
-		(layer "B.Cu")
-		(net 59)
-	)
-	(segment
-		(start 60.56 155.784814)
-		(end 61.733214 154.6116)
-		(width 0.2)
-		(layer "B.Cu")
-		(net 59)
-	)
-	(segment
-		(start 61.733214 154.6116)
+		(start 60.9052 153.6522)
 		(end 61.8646 154.6116)
 		(width 0.2)
@@
 	)
 	(segment
-		(start 56.5588 139.047072)
-		(end 56.5588 139.329914)
+		(start 56.5588 142.028273)
+		(end 57.1588 142.628273)
 		(width 0.2)
 		(layer "B.Cu")
@@
 	)
 	(segment
-		(start 60.9052 153.6522)
-		(end 61.8646 154.6116)
+		(start 60.9052 146.3756)
+		(end 60.9052 153.6522)
 		(width 0.2)
 		(layer "B.Cu")
@@
 	)
 	(segment
-		(start 56.5588 139.329914)
-		(end 59.924443 142.695557)
+		(start 60.56 155.784814)
+		(end 61.733214 154.6116)
 		(width 0.2)
 		(layer "B.Cu")
@@
 	)
 	(segment
-		(start 59.924443 142.695558)
-		(end 60.9052 143.676314)
+		(start 57.1588 142.628273)
+		(end 57.1588 142.6292)
 		(width 0.2)
 		(layer "B.Cu")
@@
 	)
 	(segment
-		(start 60.9052 143.676314)
-		(end 60.9052 153.6522)
+		(start 61.733214 154.6116)
+		(end 61.8646 154.6116)
 		(width 0.2)
 		(layer "B.Cu")
@@
 	)
 	(segment
+		(start 57.1588 142.6292)
+		(end 60.9052 146.3756)
+		(width 0.2)
+		(layer "B.Cu")
+		(net 59)
+	)
+	(segment
 		(start 48.6138 76.7404)
 		(end 46.5296 76.7404)
@@
 	)
 	(segment
-		(start 48.6138 86.2404)
-		(end 44.4468 86.2404)
+		(start 38.6556 86.2404)
+		(end 35.6132 89.2828)
 		(width 0.2)
 		(layer "B.Cu")
@@
 	)
 	(segment
-		(start 44.4468 86.2404)
-		(end 41.4044 89.2828)
+		(start 48.6138 86.2404)
+		(end 38.6556 86.2404)
 		(width 0.2)
 		(layer "B.Cu")
@@
 	)
 	(segment
-		(start 42.942 85.7404)
-		(end 41.4044 84.2028)
+		(start 37.1508 85.7404)
+		(end 35.6132 84.2028)
 		(width 0.2)
 		(layer "B.Cu")
@@
 	(segment
 		(start 48.6138 85.7404)
-		(end 42.942 85.7404)
+		(end 37.1508 85.7404)
 		(width 0.2)
 		(layer "B.Cu")
@@
 	)
 	(segment
-		(start 48.867329 92.471)
-		(end 39.1692 92.471)
+		(start 40.5408 92.471)
+		(end 38.458 94.5538)
 		(width 0.2)
 		(layer "B.Cu")
@@
 		(width 0.2)
 		(layer "B.Cu")
+		(net 158)
+	)
+	(segment
+		(start 48.867329 92.471)
+		(end 40.5408 92.471)
+		(width 0.2)
+		(layer "B.Cu")
