File: pcbs/reflow-controller-v1/temp_sensor.kicad_sch (KiCad schematic)
At the start: 7 parts, among them J1101 EB163A-04-C-180, U1101 MAX31865ATP+

Commit message: footprint assignement fixed; buzzer added
Parts:
- C1201: renamed from C1102; footprint (none) -> Capacitor_SMD:C_0603_1608Metric
- C1202: renamed from C1101; footprint (none) -> Capacitor_SMD:C_0603_1608Metric
- renumbered J1101 to J1201, R1102 to R1201, R1101 to R1202, R1103 to R1203, U1101 to U1201
Changed lines of the file:
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@@
 		(dnp no)
 		(fields_autoplaced yes)
-		(property "Reference" "R1102"
+		(property "Reference" "R1201"
 			(at 161.29 111.76 0)
 			(effects
@@
 		(dnp no)
 		(fields_autoplaced yes)
-		(property "Reference" "C1102"
+		(property "Reference" "C1201"
 			(at 124.46 58.42 0)
 			(effects
@@
 			)
 		)
-		(property "Footprint" ""
+		(property "Footprint" "Capacitor_SMD:C_0603_1608Metric"
 			(at 121.6152 63.5 0)
 			(effects
@@
 		(dnp no)
 		(fields_autoplaced yes)
-		(property "Reference" "#PWR01104"
+		(property "Reference" "#PWR01204"
 			(at 143.51 72.39 0)
 			(effects
@@
 		(dnp no)
 		(fields_autoplaced yes)
-		(property "Reference" "R1101"
+		(property "Reference" "R1202"
 			(at 167.64 82.55 0)
 			(effects
@@
 		(dnp no)
 		(fields_autoplaced yes)
-		(property "Reference" "J1101"
+		(property "Reference" "J1201"
 			(at 201.93 101.6 0)
 			(effects
@@
 		(on_board yes)
 		(dnp no)
-		(property "Reference" "U1101"
+		(property "Reference" "U1201"
 			(at 123.19 74.93 0)
 			(effects
@@
 		(dnp no)
 		(fields_autoplaced yes)
-		(property "Reference" "#PWR01103"
+		(property "Reference" "#PWR01201"
 			(at 120.65 72.39 0)
 			(effects
@@
 		(dnp no)
 		(fields_autoplaced yes)
-		(property "Reference" "C1101"
+		(property "Reference" "C1202"
 			(at 147.32 58.42 0)
 			(effects
@@
 			)
 		)
-		(property "Footprint" ""
+		(property "Footprint" "Capacitor_SMD:C_0603_1608Metric"
 			(at 144.4752 63.5 0)
 			(effects
@@
 		(dnp no)
 		(fields_autoplaced yes)
-		(property "Reference" "#PWR01101"
+		(property "Reference" "#PWR01202"
 			(at 135.89 54.61 0)
 			(effects
@@
 		(dnp no)
 		(fields_autoplaced yes)
-		(property "Reference" "#PWR01102"
+		(property "Reference" "#PWR01203"
 			(at 135.89 128.27 0)
 			(effects
@@
 		(on_board yes)
 		(dnp yes)
-		(property "Reference" "R1103"
+		(property "Reference" "R1203"
 			(at 165.1 92.71 90)
 			(effects

Commit message: add ldo for analog voltage
Connections:
- net +3V3: no longer C1202.1, U1201.20 (VDD)
- net GND: no longer R1201.2, U1201.10 (GND), U1201.16 (GND), U1201.21 (GND)
- new net +3.3VA: C1202.1, U1201.20 (VDD)
- new net GNDA: R1201.2, U1201.10 (GND), U1201.16 (GND), U1201.21 (GND)
Changed lines of the file:
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@@
 	)
 	(junction
-		(at 135.89 119.38)
+		(at 139.7 53.34)
 		(diameter 0)
 		(color 0 0 0 0)
@@
 	)
 	(junction
-		(at 135.89 53.34)
-		(diameter 0)
-		(color 0 0 0 0)
-	)
-	(junction
 		(at 138.43 119.38)
 		(diameter 0)
@@
 		(color 0 0 0 0)
 	)
-	(junction
-		(at 138.43 53.34)
-		(diameter 0)
-		(color 0 0 0 0)
+	(wire
+		(pts
+			(xy 139.7 52.07) (xy 139.7 53.34)
+		)
+		(stroke
+			(width 0)
+			(type default)
+		)
 	)
 	(wire
@@
 	(wire
 		(pts
-			(xy 133.35 111.76) (xy 133.35 119.38)
-		)
-		(stroke
-			(width 0)
-			(type default)
-		)
-	)
-	(wire
-		(pts
 			(xy 171.45 93.98) (xy 171.45 96.52)
 		)
@@
 	(wire
 		(pts
-			(xy 135.89 50.8) (xy 135.89 53.34)
+			(xy 133.35 50.8) (xy 133.35 53.34)
 		)
 		(stroke
@@
 	(wire
 		(pts
-			(xy 133.35 53.34) (xy 135.89 53.34)
-		)
-		(stroke
-			(width 0)
-			(type default)
-		)
-	)
-	(wire
-		(pts
 			(xy 151.13 104.14) (xy 194.31 104.14)
 		)
@@
 	(wire
 		(pts
+			(xy 133.35 111.76) (xy 133.35 116.84)
+		)
+		(stroke
+			(width 0)
+			(type default)
+		)
+	)
+	(wire
+		(pts
 			(xy 151.13 106.68) (xy 194.31 106.68)
 		)
@@
 	(wire
 		(pts
-			(xy 138.43 53.34) (xy 143.51 53.34)
+			(xy 138.43 53.34) (xy 139.7 53.34)
 		)
 		(stroke
@@
 	(wire
 		(pts
-			(xy 133.35 119.38) (xy 135.89 119.38)
-		)
-		(stroke
-			(width 0)
-			(type default)
-		)
-	)
-	(wire
-		(pts
 			(xy 138.43 119.38) (xy 158.75 119.38)
 		)
@@
 	(wire
 		(pts
-			(xy 135.89 119.38) (xy 138.43 119.38)
-		)
-		(stroke
-			(width 0)
-			(type default)
-		)
-	)
-	(wire
-		(pts
-			(xy 135.89 53.34) (xy 138.43 53.34)
-		)
-		(stroke
-			(width 0)
-			(type default)
-		)
-	)
-	(wire
-		(pts
 			(xy 143.51 63.5) (xy 143.51 66.04)
 		)
@@
 	(wire
 		(pts
+			(xy 139.7 53.34) (xy 143.51 53.34)
+		)
+		(stroke
+			(width 0)
+			(type default)
+		)
+	)
+	(wire
+		(pts
 			(xy 151.13 99.06) (xy 153.67 99.06)
 		)
@@
 	(wire
 		(pts
-			(xy 135.89 119.38) (xy 135.89 121.92)
+			(xy 138.43 119.38) (xy 138.43 121.92)
 		)
 		(stroke
@@
 	)
 	(symbol
-		(lib_id "power:+3V3")
-		(at 135.89 50.8 0)
+		(lib_id "power:GNDA")
+		(at 138.43 121.92 0)
 		(unit 1)
 		(exclude_from_sim no)
@@
 		(dnp no)
 		(fields_autoplaced yes)
-		(property "Reference" "#PWR01202"
-			(at 135.89 54.61 0)
-			(effects
-				(font
-					(size 1.27 1.27)
-				)
-				(hide yes)
-			)
-		)
-		(property "Value" "+3V3"
-			(at 135.89 45.72 0)
+		(property "Reference" "#PWR01106"
+			(at 138.43 128.27 0)
+			(effects
+				(font
+					(size 1.27 1.27)
+				)
+				(hide yes)
+			)
+		)
+		(property "Value" "GNDA"
+			(at 138.43 127 0)
 			(effects
 				(font
@@
 		)
 		(property "Footprint" ""
-			(at 135.89 50.8 0)
+			(at 138.43 121.92 0)
 			(effects
 				(font
@@
 		)
 		(property "Datasheet" ""
-			(at 135.89 50.8 0)
-			(effects
-				(font
-					(size 1.27 1.27)
-				)
-				(hide yes)
-			)
-		)
-		(property "Description" ""
-			(at 135.89 50.8 0)
+			(at 138.43 121.92 0)
+			(effects
+				(font
+					(size 1.27 1.27)
+				)
+				(hide yes)
+			)
+		)
+		(property "Description" "Power symbol creates a global label with name \"GNDA\" , analog ground"
+			(at 138.43 121.92 0)
 			(effects
 				(font
@@
 		)
 		(instances
-			(project "reflow-controller-v1"
+			(project ""
 				(path "/843848ae-bf49-42cb-8f8b-76790d2e568d/47b4fc3d-8fc3-490e-b9bf-4506c270c925"
-					(reference "#PWR01202")
+					(reference "#PWR01206")
 					(unit 1)
 				)
 				(path "/843848ae-bf49-42cb-8f8b-76790d2e568d/d75ecda1-c4de-4de1-8c23-afebb28677b2"
-					(reference "#PWR01101")
+					(reference "#PWR01106")
 					(unit 1)
 				)
 				(path "/843848ae-bf49-42cb-8f8b-76790d2e568d/f6f2ca5e-25e6-4058-afda-5a23263ad8e9"
-					(reference "#PWR01302")
+					(reference "#PWR01306")
 					(unit 1)
 				)
@@
 	)
 	(symbol
-		(lib_id "power:GND")
-		(at 135.89 121.92 0)
+		(lib_id "power:+3V3")
+		(at 133.35 50.8 0)
 		(unit 1)
 		(exclude_from_sim no)
@@
 		(dnp no)
 		(fields_autoplaced yes)
+		(property "Reference" "#PWR01202"
+			(at 133.35 54.61 0)
+			(effects
+				(font
+					(size 1.27 1.27)
+				)
+				(hide yes)
+			)
+		)
+		(property "Value" "+3V3"
+			(at 133.35 45.72 0)
+			(effects
+				(font
+					(size 1.27 1.27)
+				)
+			)
+		)
+		(property "Footprint" ""
+			(at 133.35 50.8 0)
+			(effects
+				(font
+					(size 1.27 1.27)
+				)
+				(hide yes)
+			)
+		)
+		(property "Datasheet" ""
+			(at 133.35 50.8 0)
+			(effects
+				(font
+					(size 1.27 1.27)
+				)
+				(hide yes)
+			)
+		)
+		(property "Description" ""
+			(at 133.35 50.8 0)
+			(effects
+				(font
+					(size 1.27 1.27)
+				)
+				(hide yes)
+			)
+		)
+		(pin "1"
+		)
+		(instances
+			(project "reflow-controller-v1"
+				(path "/843848ae-bf49-42cb-8f8b-76790d2e568d/47b4fc3d-8fc3-490e-b9bf-4506c270c925"
+					(reference "#PWR01202")
+					(unit 1)
+				)
+				(path "/843848ae-bf49-42cb-8f8b-76790d2e568d/d75ecda1-c4de-4de1-8c23-afebb28677b2"
+					(reference "#PWR01101")
+					(unit 1)
+				)
+				(path "/843848ae-bf49-42cb-8f8b-76790d2e568d/f6f2ca5e-25e6-4058-afda-5a23263ad8e9"
+					(reference "#PWR01302")
+					(unit 1)
+				)
+			)
+		)
+	)
+	(symbol
+		(lib_id "power:+3.3VA")
+		(at 139.7 52.07 0)
+		(unit 1)
+		(exclude_from_sim no)
+		(in_bom yes)
+		(on_board yes)
+		(dnp no)
+		(fields_autoplaced yes)
+		(property "Reference" "#PWR01105"
+			(at 139.7 55.88 0)
+			(effects
+				(font
+					(size 1.27 1.27)
+				)
+				(hide yes)
+			)
+		)
+		(property "Value" "+3.3VA"
+			(at 139.7 46.99 0)
+			(effects
+				(font
+					(size 1.27 1.27)
+				)
+			)
+		)
+		(property "Footprint" ""
+			(at 139.7 52.07 0)
+			(effects
+				(font
+					(size 1.27 1.27)
+				)
+				(hide yes)
+			)
+		)
+		(property "Datasheet" ""
+			(at 139.7 52.07 0)
+			(effects
+				(font
+					(size 1.27 1.27)
+				)
+				(hide yes)
+			)
+		)
+		(property "Description" "Power symbol creates a global label with name \"+3.3VA\""
+			(at 139.7 52.07 0)
+			(effects
+				(font
+					(size 1.27 1.27)
+				)
+				(hide yes)
+			)
+		)
+		(pin "1"
+		)
+		(instances
+			(project ""
+				(path "/843848ae-bf49-42cb-8f8b-76790d2e568d/47b4fc3d-8fc3-490e-b9bf-4506c270c925"
+					(reference "#PWR01205")
+					(unit 1)
+				)
+				(path "/843848ae-bf49-42cb-8f8b-76790d2e568d/d75ecda1-c4de-4de1-8c23-afebb28677b2"
+					(reference "#PWR01105")
+					(unit 1)
+				)
+				(path "/843848ae-bf49-42cb-8f8b-76790d2e568d/f6f2ca5e-25e6-4058-afda-5a23263ad8e9"
+					(reference "#PWR01305")
+					(unit 1)
+				)
+			)
+		)
+	)
+	(symbol
+		(lib_id "power:GND")
+		(at 133.35 116.84 0)
+		(unit 1)
+		(exclude_from_sim no)
+		(in_bom yes)
+		(on_board yes)
+		(dnp no)
+		(fields_autoplaced yes)
 		(property "Reference" "#PWR01203"
-			(at 135.89 128.27 0)
+			(at 133.35 123.19 0)
 			(effects
 				(font
@@
 		)
 		(property "Value" "GND"
-			(at 135.89 127 0)
+			(at 133.35 121.92 0)
 			(effects
 				(font
@@
 		)
 		(property "Footprint" ""
-			(at 135.89 121.92 0)
+			(at 133.35 116.84 0)
 			(effects
 				(font
@@
 		)
 		(property "Datasheet" ""
-			(at 135.89 121.92 0)
+			(at 133.35 116.84 0)
 			(effects
 				(font
@@
 		)
 		(property "Description" ""
-			(at 135.89 121.92 0)
-			(effects
-				(font
+			(at 133.35 116.84 0)
+			(effects
+				(font

Commit message: update analog voltage ldo placement&routing
Connections:
- net GNDA is gone; now on net GND: R1201.2, U1201.10 (GND), U1201.16 (GND), U1201.21 (GND)
Changed lines of the file:
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@@
+	(wire
+		(pts
+			(xy 133.35 119.38) (xy 138.43 119.38)
+		)
+		(stroke
+			(width 0)
+			(type default)
+		)
+	)
 	(wire
 		(pts
@@
 	(wire
 		(pts
-			(xy 133.35 111.76) (xy 133.35 116.84)
+			(xy 133.35 111.76) (xy 133.35 119.38)
 		)
 		(stroke
@@
 			)
 			(justify right)
+		)
+	)
+	(symbol
+		(lib_name "GND_1")
+		(lib_id "power:GND")
+		(at 138.43 121.92 0)
+		(unit 1)
+		(exclude_from_sim no)
+		(in_bom yes)
+		(on_board yes)
+		(dnp no)
+		(fields_autoplaced yes)
+		(property "Reference" "#PWR01102"
+			(at 138.43 128.27 0)
+			(effects
+				(font
+					(size 1.27 1.27)
+				)
+				(hide yes)
+			)
+		)
+		(property "Value" "GND"
+			(at 138.43 127 0)
+			(effects
+				(font
+					(size 1.27 1.27)
+				)
+			)
+		)
+		(property "Footprint" ""
+			(at 138.43 121.92 0)
+			(effects
+				(font
+					(size 1.27 1.27)
+				)
+				(hide yes)
+			)
+		)
+		(property "Datasheet" ""
+			(at 138.43 121.92 0)
+			(effects
+				(font
+					(size 1.27 1.27)
+				)
+				(hide yes)
+			)
+		)
+		(property "Description" "Power symbol creates a global label with name \"GND\" , ground"
+			(at 138.43 121.92 0)
+			(effects
+				(font
+					(size 1.27 1.27)
+				)
+				(hide yes)
+			)
+		)
+		(pin "1"
+		)
+		(instances
+			(project ""
+				(path "/843848ae-bf49-42cb-8f8b-76790d2e568d/47b4fc3d-8fc3-490e-b9bf-4506c270c925"
+					(reference "#PWR01203")
+					(unit 1)
+				)
+				(path "/843848ae-bf49-42cb-8f8b-76790d2e568d/d75ecda1-c4de-4de1-8c23-afebb28677b2"
+					(reference "#PWR01102")
+					(unit 1)
+				)
+				(path "/843848ae-bf49-42cb-8f8b-76790d2e568d/f6f2ca5e-25e6-4058-afda-5a23263ad8e9"
+					(reference "#PWR01303")
+					(unit 1)
+				)
+			)
 		)
 	)
@@
 	)
 	(symbol
-		(lib_id "power:GNDA")
-		(at 138.43 121.92 0)
-		(unit 1)
-		(exclude_from_sim no)
-		(in_bom yes)
-		(on_board yes)
-		(dnp no)
-		(fields_autoplaced yes)
-		(property "Reference" "#PWR01106"
-			(at 138.43 128.27 0)
-			(effects
-				(font
-					(size 1.27 1.27)
-				)
-				(hide yes)
-			)
-		)
-		(property "Value" "GNDA"
-			(at 138.43 127 0)
-			(effects
-				(font
-					(size 1.27 1.27)
-				)
-			)
-		)
-		(property "Footprint" ""
-			(at 138.43 121.92 0)
-			(effects
-				(font
-					(size 1.27 1.27)
-				)
-				(hide yes)
-			)
-		)
-		(property "Datasheet" ""
-			(at 138.43 121.92 0)
-			(effects
-				(font
-					(size 1.27 1.27)
-				)
-				(hide yes)
-			)
-		)
-		(property "Description" "Power symbol creates a global label with name \"GNDA\" , analog ground"
-			(at 138.43 121.92 0)
-			(effects
-				(font
-					(size 1.27 1.27)
-				)
-				(hide yes)
-			)
-		)
-		(pin "1"
-		)
-		(instances
-			(project ""
-				(path "/843848ae-bf49-42cb-8f8b-76790d2e568d/47b4fc3d-8fc3-490e-b9bf-4506c270c925"
-					(reference "#PWR01206")
-					(unit 1)
-				)
-				(path "/843848ae-bf49-42cb-8f8b-76790d2e568d/d75ecda1-c4de-4de1-8c23-afebb28677b2"
-					(reference "#PWR01106")
-					(unit 1)
-				)
-				(path "/843848ae-bf49-42cb-8f8b-76790d2e568d/f6f2ca5e-25e6-4058-afda-5a23263ad8e9"
-					(reference "#PWR01306")
-					(unit 1)
-				)
-			)
-		)
-	)
-	(symbol
 		(lib_id "power:+3V3")
 		(at 133.35 50.8 0)
@@
 		(dnp no)
 		(fields_autoplaced yes)
-		(property "Reference" "#PWR01105"
+		(property "Reference" "#PWR01205"
 			(at 139.7 55.88 0)
 			(effects
@@
 					(unit 1)
 				)
-			)
-		)
-	)
-	(symbol
-		(lib_id "power:GND")
-		(at 133.35 116.84 0)
-		(unit 1)
-		(exclude_from_sim no)
-		(in_bom yes)
-		(on_board yes)
-		(dnp no)
-		(fields_autoplaced yes)
-		(property "Reference" "#PWR01203"
-			(at 133.35 123.19 0)
-			(effects
-				(font
-					(size 1.27 1.27)
-				)
-				(hide yes)
-			)
-		)
-		(property "Value" "GND"
-			(at 133.35 121.92 0)
-			(effects
-				(font
-					(size 1.27 1.27)
-				)
-			)
-		)
-		(property "Footprint" ""
-			(at 133.35 116.84 0)
-			(effects
-				(font
-					(size 1.27 1.27)
-				)
-				(hide yes)
-			)
-		)
-		(property "Datasheet" ""
-			(at 133.35 116.84 0)
-			(effects
-				(font
-					(size 1.27 1.27)
-				)
-				(hide yes)
-			)
-		)
-		(property "Description" ""
-			(at 133.35 116.84 0)
-			(effects
-				(font
-					(size 1.27 1.27)
-				)
-				(hide yes)
-			)
-		)
-		(pin "1"
-		)
-		(instances
-			(project "reflow-controller-v1"
-				(path "/843848ae-bf49-42cb-8f8b-76790d2e568d/47b4fc3d-8fc3-490e-b9bf-4506c270c925"
-					(reference "#PWR01203")
-					(unit 1)
-				)
-				(path "/843848ae-bf49-42cb-8f8b-76790d2e568d/d75ecda1-c4de-4de1-8c23-afebb28677b2"
-					(reference "#PWR01102")
-					(unit 1)
-				)
-				(path "/843848ae-bf49-42cb-8f8b-76790d2e568d/f6f2ca5e-25e6-4058-afda-5a23263ad8e9"
-					(reference "#PWR01303")
-					(unit 1)
-				)
