File: pcbs/reflow-controller-v1/common/pcb_interconnect.kicad_sch (KiCad schematic)
At the start: 2 parts, among them J801 Power, J802 Data

Commit message: route hv pcb
Connections:
- net SSR1: now also J802.5 (Pin_5); no longer J802.1 (Pin_1)
- net SSR2: now also J802.4 (Pin_4); no longer J802.2 (Pin_2)
- net SSR4: now also J802.2 (Pin_2); no longer J802.4 (Pin_4)
- net Zero: now also J802.1 (Pin_1); no longer J802.5 (Pin_5)
- net +3.3V renamed +3V3
Changed lines of the file:
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@@
 	(hierarchical_label "SSR2"
 		(shape bidirectional)
-		(at 163.83 97.79 0)
+		(at 163.83 102.87 0)
 		(effects
 			(font
@@
 	(hierarchical_label "SSR4"
 		(shape bidirectional)
-		(at 163.83 102.87 0)
+		(at 163.83 97.79 0)
 		(effects
 			(font
@@
 	(hierarchical_label "Zero"
 		(shape bidirectional)
-		(at 163.83 105.41 0)
+		(at 163.83 95.25 0)
 		(effects
 			(font
@@
 	(hierarchical_label "SSR1"
 		(shape bidirectional)
-		(at 163.83 95.25 0)
+		(at 163.83 105.41 0)
 		(effects
 			(font
@@
 	)
 	(symbol
-		(lib_id "power:+3.3V")
+		(lib_id "power:+3V3")
 		(at 166.37 68.58 0)
 		(unit 1)
@@
 		(dnp no)
 		(fields_autoplaced yes)
-		(property "Reference" "#PWR0804"
+		(property "Reference" "#PWR0805"
 			(at 166.37 72.39 0)
 			(effects
@@
 			)
 		)
-		(property "Value" "+3.3V"
+		(property "Value" "+3V3"
 			(at 166.37 63.5 0)
 			(effects
@@
 			)
 		)
-		(property "Description" "Power symbol creates a global label with name \"+3.3V\""
+		(property "Description" "Power symbol creates a global label with name \"+3V3\""
 			(at 166.37 68.58 0)
 			(effects
@@
 		)
 		(instances
-			(project "ui"
-				(path "/2ced3b3e-2fc8-4776-88d1-4bcb3cd16514/f84f6660-f8eb-481a-b914-aee57f214b58"
-					(reference "#PWR0204")
-					(unit 1)
-				)
-			)
 			(project ""
-				(path "/843848ae-bf49-42cb-8f8b-76790d2e568d/70a6fcff-45f3-4adb-97e9-6ae77cc29097"
-					(reference "#PWR01702")
-					(unit 1)
-				)
-			)
-			(project "hv"
 				(path "/bfc257b6-4a03-4e6b-b2e0-eeb653e202b4/32264195-0edd-4756-a40a-d0c1061e5db1"
-					(reference "#PWR0804")
-					(unit 1)
-				)
+					(reference "#PWR0805")
+					(unit 1)
+				)
