File: pcbs/reflow-controller-v1/hv/ac-dc-converter.kicad_sch (KiCad schematic)
At the start: 3 parts

Commit message: improve component selection
Parts:
- C201: Order (none) -> Würth 885012205018
- C202: value EEEFK1E470P -> 47μF; Order (none) -> Würth 865060343004
Other:
- note removed: "47µF"
Changed lines of the file:
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@@
 	(generator_version "9.0")
 	(paper "A4")
-	(text "47µF"
-		(exclude_from_sim no)
-		(at 163.83 43.18 0)
-		(effects
-			(font
-				(size 1.27 1.27)
-			)
-			(justify left bottom)
-		)
-	)
 	(junction
 		(at 160.02 33.02)
@@
 		(on_board yes)
 		(dnp no)
-		(fields_autoplaced yes)
 		(property "Reference" "C201"
 			(at 144.78 38.1 0)
@@
 			)
 		)
-		(property "Datasheet" "~"
+		(property "Datasheet" "https://www.we-online.com/components/products/datasheet/885012205018.pdf"
 			(at 140.97 39.37 0)
 			(effects
@@
 				)
 				(hide yes)
+			)
+		)
+		(property "Order" "Würth 885012205018"
+			(at 144.78 42.672 0)
+			(effects
+				(font
+					(size 1.27 1.27)
+				)
+				(justify left)
 			)
 		)
@@
 		(on_board yes)
 		(dnp no)
-		(fields_autoplaced yes)
 		(property "Reference" "C202"
-			(at 163.83 37.211 0)
-			(effects
-				(font
-					(size 1.27 1.27)
-				)
-				(justify left)
-			)
-		)
-		(property "Value" "EEEFK1E470P"
-			(at 163.83 39.751 0)
+			(at 163.83 37.2109 0)
+			(effects
+				(font
+					(size 1.27 1.27)
+				)
+				(justify left)
+			)
+		)
+		(property "Value" "47μF"
+			(at 163.83 39.7509 0)
 			(effects
 				(font
@@
 			)
 		)
-		(property "Datasheet" "~"
+		(property "Datasheet" "https://www.we-online.com/components/products/datasheet/865060343004.pdf"
 			(at 160.02 39.37 0)
 			(effects
@@
 			)
 		)
+		(property "Order" "Würth 865060343004"
+			(at 163.83 41.91 0)
+			(effects
+				(font
+					(size 1.27 1.27)
+				)
+				(justify left)
+			)
+		)
