File: pcbs/reflow-controller-v1/hv/ssr.kicad_sch (KiCad schematic)
At the start: 7 parts, among them U301 MOC3043SM

Commit message: split pcbs into two for safety
Parts:
- removed D301: T1620T-8G-TR, Package_TO_SOT_SMD:TO-263-2, symbol Device:Q_TRIAC_A1A2G
- added D301: T1620T-8G-TR, Package_TO_SOT_SMD:TO-263-2, symbol Triac_Thyristor:Generic_Triac_A1A2G
- renumbered R304 to R302, R302 to R303, R305 to R304
Connections:
- net MAIN: now also D301.2 (A2)
- net MAIN_OUT: now also D301.1 (A1)
- net at R302.1, U301.4: now also D301.3 (G)

Commit message: improve component selection
Parts:
- R301: value 180 -> 180Ω; Order (none) -> Würth 560112116097
- R302: value 330 -> 330Ω
- R303: value 360 -> 360Ω
Changed lines of the file:
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@@
+		)
+	)
+	(rule_area
+		(polyline
+			(pts
+				(xy 88.9 73.66) (xy 88.9 102.87) (xy 132.08 102.87) (xy 132.08 73.66)
+			)
+			(stroke
+				(width 0)
+				(type dash)
+			)
+			(fill
+				(type none)
+			)
+		)
+	)
+	(netclass_flag ""
+		(length 2.54)
+		(shape round)
+		(at 109.22 73.66 0)
+		(fields_autoplaced yes)
+		(effects
+			(font
+				(size 1.27 1.27)
+			)
+			(justify left bottom)
+		)
+		(property "Netclass" "LV"
+			(at 109.9185 71.12 0)
+			(effects
+				(font
+					(size 1.27 1.27)
+				)
+				(justify left)
+			)
+		)
+		(property "Component Class" ""
+			(at -52.07 -11.43 0)
+			(effects
+				(font
+					(size 1.27 1.27)
+					(italic yes)
+				)
+			)
 		)
 	)
@@
 			)
 		)
-		(property "Datasheet" "~"
+		(property "Datasheet" "https://www.st.com/resource/en/datasheet/t1620t-8g.pdf"
 			(at 172.72 95.25 90)
 			(effects
@@
 			)
 		)
-		(property "Value" "330"
+		(property "Value" "330Ω"
 			(at 154.94 105.41 0)
 			(effects
@@
 			)
 		)
-		(property "Value" "180"
+		(property "Value" "180Ω"
 			(at 118.11 83.82 90)
 			(effects
@@
 			)
 		)
-		(property "Datasheet" "~"
+		(property "Datasheet" "https://www.we-online.com/components/products/datasheet/560112116097.pdf"
 			(at 118.11 87.63 0)
 			(effects
@@
 		(property "Description" "Resistor"
 			(at 118.11 87.63 0)
+			(effects
+				(font
+					(size 1.27 1.27)
+				)
+				(hide yes)
+			)
+		)
+		(property "Order" "Würth 560112116097"
+			(at 118.11 87.63 90)
 			(effects
 				(font
@@
 			)
 		)
-		(property "Value" "360"
+		(property "Value" "360Ω"
 			(at 158.75 83.82 90)
 			(effects
